Commit message: Random Snake

File: body.urdf (robot description, URDF)
Before this commit: robot robot, 5 links, 4 joints
Links:
- removed link Backleg
- removed link Frontleg
- removed link Leftleg
- removed link Rightleg
- removed link Torso
- added link Head, mass 1; collision box size=1 4 2; visual box size=1 4 2
- added link Link0, mass 1; collision box size=1 1 4; visual box size=1 1 4
- added link Link1, mass 1; collision box size=4 3 1; visual box size=4 3 1
- added link Link2, mass 1; collision box size=4 5 4; visual box size=4 5 4
- added link Link3, mass 1; collision box size=4 2 5; visual box size=4 2 5
- added link Link4, mass 1; collision box size=4 5 2; visual box size=4 5 2
- added link Link5, mass 1; collision box size=4 5 5; visual box size=4 5 5
- added link Link6, mass 1; collision box size=5 3 3; visual box size=5 3 3
Joints:
- removed joint Torso_Backleg
- removed joint Torso_Frontleg
- removed joint Torso_Leftleg
- removed joint Torso_Rightleg
- added joint Head_Link0: type revolute, parent Head, child Link0, origin xyz=-10 18.0 2.5 rpy=0 0 0, axis 0 0 1, limit lower=-3.14159 upper=3.14159 effort=0.0 velocity=0.0
- added joint Link0_Link1: type revolute, parent Link0, child Link1, origin xyz=0 -1 0 rpy=0 0 0, axis 0 0 1, limit lower=-3.14159 upper=3.14159 effort=0.0 velocity=0.0
- added joint Link1_Link2: type revolute, parent Link1, child Link2, origin xyz=0 -3 0 rpy=0 0 0, axis 0 0 1, limit lower=-3.14159 upper=3.14159 effort=0.0 velocity=0.0
- added joint Link2_Link3: type revolute, parent Link2, child Link3, origin xyz=0 -5 0 rpy=0 0 0, axis 0 0 1, limit lower=-3.14159 upper=3.14159 effort=0.0 velocity=0.0
- added joint Link3_Link4: type revolute, parent Link3, child Link4, origin xyz=0 -2 0 rpy=0 0 0, axis 0 0 1, limit lower=-3.14159 upper=3.14159 effort=0.0 velocity=0.0
- added joint Link4_Link5: type revolute, parent Link4, child Link5, origin xyz=0 -5 0 rpy=0 0 0, axis 0 0 1, limit lower=-3.14159 upper=3.14159 effort=0.0 velocity=0.0
- added joint Link5_Link6: type revolute, parent Link5, child Link6, origin xyz=0 -5 0 rpy=0 0 0, axis 0 0 1, limit lower=-3.14159 upper=3.14159 effort=0.0 velocity=0.0

Commit message: Update 2/14

File: body.urdf (robot description, URDF)
Before this commit: robot robot, 8 links, 7 joints
Links:
- removed link Head
- removed link Link4
- removed link Link5
- removed link Link6
- link Link0: geometry collision box size=0.7934475894017761 0.8095176747178948 0.7975469418093027; visual box size=0.7934475894017761 0.8095176747178948 0.7975469418093027
- link Link1: geometry collision box size=0.18542707145667991 0.749936684461131 0.5003290211387642; visual box size=0.18542707145667991 0.749936684461131 0.5003290211387642
- link Link2: geometry collision box size=0.08805621961752175 0.07042512230518305 0.2705482273812503; visual box size=0.08805621961752175 0.07042512230518305 0.2705482273812503
- link Link3: geometry collision box size=0.1976532396971713 0.17240539810837674 0.86434497572423; visual box size=0.1976532396971713 0.17240539810837674 0.86434497572423
Joints:
- removed joint Head_Link0
- removed joint Link3_Link4
- removed joint Link4_Link5
- removed joint Link5_Link6
- joint Link0_Link1: axis 0 0 1 -> 0.03981546366889044 0.9837059795859147 0.47853760169069737; origin xyz=0 -1 0 rpy=0 0 0 -> xyz=-0.39672379470088803 0 0 rpy=0 0 0
- joint Link1_Link2: axis 0 0 1 -> 0.5864853968680906 0.12737873564010183 0.723060586569856; origin xyz=0 -3 0 rpy=0 0 0 -> xyz=-0.09271353572833996 0.3749683422305655 0 rpy=0 0 0
- joint Link2_Link3: axis 0 0 1 -> 0.5069417605709553 0.44497441220297074 0.9072537616989708; origin xyz=0 -5 0 rpy=0 0 0 -> xyz=0 0.07042512230518305 0 rpy=0 0 0
